File: PCM3128.kicad_pcb (KiCad board)
At the start: 2 copper layers, 84 x 100 mm, 36 parts, among them IC1 TPA3128, J1 IN, J2 IN 1, J3 IN 2, K1 G6K-2P-Y_DC3, K2 G6K-2P-Y_DC3, U1 LMR51430, U4 ULN2003

Commit message: lots of work
Parts:
- added C17: 220nF, Capacitor_THT:C_Rect_L7.2mm_W2.5mm_P5.00mm_FKS2_FKP2_MKS2_MKP2, F.Cu at (214.8, 62.3)
- added C18: 220nF, Capacitor_THT:C_Rect_L7.2mm_W2.5mm_P5.00mm_FKS2_FKP2_MKS2_MKP2, F.Cu at (214.8, 66.3)
- added C19: 220nF, Capacitor_THT:C_Rect_L7.2mm_W2.5mm_P5.00mm_FKS2_FKP2_MKS2_MKP2, F.Cu at (159.4, 105.4)
- added C20: 220nF, Capacitor_THT:C_Rect_L7.2mm_W2.5mm_P5.00mm_FKS2_FKP2_MKS2_MKP2, F.Cu at (165.8, 99.1)
- added L2: 10uH, Custom:ETQP5M100YFC, F.Cu at (204.6, 67.0)
- added L3: 10uH, Custom:ETQP5M100YFC, F.Cu at (204.6, 80.4)
- added L4: 10uH, Custom:ETQP5M100YFC, F.Cu at (204.6, 93.9)
- added L5: 10uH, Custom:ETQP5M100YFC, F.Cu at (204.6, 107.3)
- moved C9 64.2 mm to (79.7, 132.4)
- moved C14 64.2 mm to (79.7, 135.7)
- moved C16 64.2 mm to (79.7, 139.1)
- moved C7 64.2 mm to (79.7, 125.7)
- moved C8 64.2 mm to (79.7, 129.0)
- moved C11 33.1 mm to (176.0, 119.5)
- moved C12 33.1 mm to (177.5, 119.5)
- moved C10 33.1 mm to (174.5, 119.5)
- moved C13 28.4 mm to (145.8, 113.5)
- moved C15 28.4 mm to (144.3, 113.5)
- moved G*** 24.5 mm to (151.1, 164.5)
- moved C25 22.3 mm to (150.4, 137.1)
- moved C26 22.3 mm to (156.5, 137.1)
- moved C27 22.3 mm to (168.7, 137.1)
- moved C28 22.3 mm to (162.6, 137.1)
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Connections:
- IC1 pad 20: unconnected-(IC1-BSNL-Pad20) -> /BSNL
- IC1 pad 21: unconnected-(IC1-OUTNL-Pad21) -> /OUTNL
- IC1 pad 23: unconnected-(IC1-OUTPL-Pad23) -> /OUTPL
- IC1 pad 24: unconnected-(IC1-BSPL-Pad24) -> /BSPL
- IC1 pad 26: unconnected-(IC1-BSNR-Pad26) -> /BSNR
- IC1 pad 27: unconnected-(IC1-OUTNR-Pad27) -> /OUTNR
- IC1 pad 29: unconnected-(IC1-OUTPR-Pad29) -> /OUTPR
- IC1 pad 30: unconnected-(IC1-BSPR-Pad30) -> /BSPR
Routing:
- net /PVCC: track 13.3 -> 0.00 mm
- net Net-(IC1-AVCC): track 3.39 -> 0.00 mm
