File: PCM3128.kicad_sch (KiCad schematic)
At the start: 35 parts, among them IC1 TPA3128, J1 IN, J2 IN 1, J3 IN 2, K1 G6K-2P-Y_DC3, K2 G6K-2P-Y_DC3, U1 LMR51430, U4 ULN2003

Commit message: lots of work
Parts:
- added C17, C18, C19, C20: 220nF, Capacitor_THT:C_Rect_L7.2mm_W2.5mm_P5.00mm_FKS2_FKP2_MKS2_MKP2, symbol Device:C
- added L2, L3, L4, L5: 10uH, Custom:ETQP5M100YFC, symbol Device:L
Connections:
- net BSNL: now reaches IC1.20 (BSNL)
- net BSNL: now also C20.1
- net OUTNL: now reaches IC1.21 (OUTNL)
- net OUTNL: now also C20.2, L4.1
- net OUTPL: now reaches IC1.23 (OUTPL)
- net OUTPL: now also C19.2, L3.1
- net BSPL: now reaches IC1.24 (BSPL)
- net BSPL: now also C19.1
- net BSNR: now reaches IC1.26 (BSNR)
- net BSNR: now also C18.1
- net OUTNR: now reaches IC1.27 (OUTNR)
- net OUTNR: now also C18.2, L2.1
- net OUTPR: now reaches IC1.29 (OUTPR)
- net OUTPR: now also C17.2, L5.1
- net BSPR: now reaches IC1.30 (BSPR)
- net BSPR: now also C17.1
Other:
- moved on the sheet: C10, C11, C12, C13, C14, C15, C16, C25, C26, C27, C28, C7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
