File: TPA3250/TPA3250.kicad_pcb (KiCad board)
At the start: 4 copper layers, 173.7 x 66.3 mm, 176 parts, among them IC3 TPS65133, J1 L +, J2 L -, J3 R +, J4 R -, J5 IN, J6 PROG, J7 24V IN, J8 GND, J9 VOL, Q1 DMP4015SK3, U1 TPA3250, U2 ATtiny1614-SS, U3 LMR51430, U4 OPA1656ID, U5 OPA1656ID, U6 LM4562, U7 PGA2311, U8 LMR51430

Commit message: more work
Parts:
- added C88: 1uF, Capacitor_SMD:C_1206_3216Metric_Pad1.33x1.80mm_HandSolder, F.Cu at (213.1, 95.2)
- added C88: 1uF, Capacitor_SMD:C_1206_3216Metric_Pad1.33x1.80mm_HandSolder, F.Cu at (213.1, 109.7)
- added C89: 1uF, Capacitor_SMD:C_1206_3216Metric_Pad1.33x1.80mm_HandSolder, F.Cu at (274.4, 131.7)
- added C90: 1uF, Capacitor_SMD:C_1206_3216Metric_Pad1.33x1.80mm_HandSolder, F.Cu at (274.4, 135.1)
- added C91: 1uF, Capacitor_SMD:C_1206_3216Metric_Pad1.33x1.80mm_HandSolder, F.Cu at (213.9, 107.2)
- added C91: 1uF, Capacitor_SMD:C_1206_3216Metric_Pad1.33x1.80mm_HandSolder, F.Cu at (213.9, 97.8)
- added C92: 1000uF, Capacitor_THT:CP_Radial_D12.5mm_P5.00mm, F.Cu at (215.1, 123.7)
- added C93: 1000uF, Capacitor_THT:CP_Radial_D12.5mm_P5.00mm, F.Cu at (215.1, 81.2)
- moved J5 242.9 mm to (258.8, 155.7), turned to 90 degrees
- moved C22 238.3 mm to (251.2, 149.9), turned to 90 degrees
- moved C21 233.1 mm to (251.2, 156.5), turned to -90 degrees
- moved C23 232.4 mm to (242.3, 144.8), turned to 0 degrees
- moved R9 230.7 mm to (242.3, 146.8), turned to 0 degrees
- moved C25 227.7 mm to (244.3, 153.2), turned to 90 degrees
- moved U6 226.5 mm to (240.5, 149.4), turned to -90 degrees
- moved R7 226.0 mm to (236.5, 144.8), turned to 0 degrees
- moved R5 224.2 mm to (236.5, 146.8), turned to 180 degrees
- moved R11 217.9 mm to (228.9, 144.7), turned to 180 degrees
- moved R10 217.0 mm to (239.5, 159.5), turned to 0 degrees
- moved C24 215.4 mm to (239.5, 161.5), turned to 0 degrees
- moved F1 211.9 mm to (248.8, 47.4), turned to 180 degrees
- moved R6 210.5 mm to (233.9, 159.5), turned to 180 degrees
- moved R8 208.9 mm to (233.9, 161.5), turned to 0 degrees
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Connections:
- U1 pad V: (no net) -> GND
Routing:
- net Net-(U7-V_{OUT}L): track 0.00 -> 83.1 mm
- net /SUM_B: track 3.32 -> 70.8 mm, vias 0 -> 1
- net Net-(C19-Pad1): track 0.00 -> 65.8 mm, vias 0 -> 1
- net Net-(C20-Pad1): track 0.00 -> 40.7 mm, vias 0 -> 1
- net /SUM_A: track 5.05 -> 45.6 mm, vias 0 -> 1
- net Net-(F1-Pad1): track 0.00 -> 11.4 mm
- net Net-(C13-Pad1): track 43.9 -> 49.6 mm
- net Net-(C12-Pad2): track 44.0 -> 49.8 mm
- net Net-(C11-Pad1): track 43.8 -> 49.4 mm
- net Net-(C1-Pad2): track 43.2 -> 48.8 mm
- net Net-(C55-Pad2): track 0.00 -> 5.19 mm
- net Net-(C52-Pad2): track 0.00 -> 5.06 mm
- net Net-(C50-Pad1): track 0.00 -> 5.05 mm
- net Net-(C54-Pad2): track 0.00 -> 3.78 mm
- net /PVDD_24V: vias 0 -> 16
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- added copper zone on F.Cu, net /PVDD_24V
- added copper zone on In2.Cu, net /PVDD_24V
Other:
- board size 173.7 x 66.3 mm -> 130 x 130 mm

Commit message: more work
Parts:
- removed the C43 at (45.8, 65.7)
- removed the C43 at (115.1, 134.0)
- removed G***: LOGO, Custom:LOGONEW
- removed J7: 24V IN, Spade connector:TE_62409-1
- removed J8: GND, Spade connector:TE_62409-1
- removed J9: VOL, Connector_JST:JST_XH_B3B-XH-A_1x03_P2.50mm_Vertical
- removed the R33 at (119.1, 68.3)
- removed the R33 at (32.1, 56.6)
- removed the R34 at (119.1, 71.2)
- removed the R34 at (32.1, 59.5)
- removed the R36 at (32.1, 62.5)
- removed the R36 at (278.7, 87.3)
- removed the R37 at (55.7, 56.8)
- removed the R37 at (278.7, 90.3)
- removed the R40 at (117.6, 89.9)
- removed the R40 at (181.2, 69.6)
- removed the R41 at (36.8, 56.6)
- removed the R41 at (283.5, 87.3)
- added C100: 10uF, Capacitor_SMD:C_0805_2012Metric_Pad1.18x1.45mm_HandSolder, F.Cu at (75.9, 188.3)
- added C101: 10nF, Capacitor_SMD:C_0805_2012Metric_Pad1.18x1.45mm_HandSolder, F.Cu at (93.8, 149.2)
- added C102: 220uF, Capacitor_THT:CP_Radial_D6.3mm_P2.50mm, F.Cu at (68.4, 185.5)
- added C103: 10uF, Capacitor_SMD:C_1206_3216Metric_Pad1.33x1.80mm_HandSolder, F.Cu at (88.4, 152.8)
- added C104: 100nF, Capacitor_SMD:C_1206_3216Metric_Pad1.33x1.80mm_HandSolder, F.Cu at (62.5, 178.8)
- added C105: 10uF, Capacitor_SMD:C_1206_3216Metric_Pad1.33x1.80mm_HandSolder, F.Cu at (62.5, 182.1)
- added C106: 1uF, Capacitor_SMD:C_1206_3216Metric_Pad1.33x1.80mm_HandSolder, F.Cu at (62.5, 185.4)
- added C107: 100nF, Capacitor_SMD:C_1206_3216Metric_Pad1.33x1.80mm_HandSolder, F.Cu at (62.5, 188.8)
- added C108: 100nF, Capacitor_SMD:C_1206_3216Metric_Pad1.33x1.80mm_HandSolder, F.Cu at (88.4, 156.1)
- added C109: 100nF, Capacitor_SMD:C_1206_3216Metric_Pad1.33x1.80mm_HandSolder, F.Cu at (88.4, 159.4)
- added C110: 2.2uF, Capacitor_SMD:C_0805_2012Metric_Pad1.18x1.45mm_HandSolder, F.Cu at (200.6, 168.9)
- added C111: 2.2uF, Capacitor_SMD:C_0805_2012Metric_Pad1.18x1.45mm_HandSolder, F.Cu at (196.0, 172.6)
- added C112: 10uF, Capacitor_SMD:C_0805_2012Metric_Pad1.18x1.45mm_HandSolder, F.Cu at (93.8, 158.3)
- added C113: 100nF, Capacitor_SMD:C_1206_3216Metric_Pad1.33x1.80mm_HandSolder, F.Cu at (101.9, 181.2)
- added C114: 1uF, Capacitor_SMD:C_1206_3216Metric_Pad1.33x1.80mm_HandSolder, F.Cu at (101.9, 184.5)
- added C115: 10nF, Capacitor_SMD:C_0805_2012Metric_Pad1.18x1.45mm_HandSolder, F.Cu at (93.8, 161.3)
- added C116: 10uF, Capacitor_SMD:C_1206_3216Metric_Pad1.33x1.80mm_HandSolder, F.Cu at (88.4, 169.5)
- added C117: 2.2nF, Capacitor_SMD:C_0805_2012Metric_Pad1.18x1.45mm_HandSolder, F.Cu at (188.8, 173.5)
- added C118: 2.2nF, Capacitor_SMD:C_0805_2012Metric_Pad1.18x1.45mm_HandSolder, F.Cu at (188.8, 177.4)
- added C119: 100nF, Capacitor_SMD:C_1206_3216Metric_Pad1.33x1.80mm_HandSolder, F.Cu at (242.4, 176.5)
- added C43: 1uF, Capacitor_THT:C_Rect_L7.2mm_W5.5mm_P5.00mm_FKS2_FKP2_MKS2_MKP2, F.Cu at (168.9, 107.2)
- added C94: 1uF, Capacitor_SMD:C_1206_3216Metric_Pad1.33x1.80mm_HandSolder, F.Cu at (94.5, 69.2)
- added C95: 1uF, Capacitor_SMD:C_1206_3216Metric_Pad1.33x1.80mm_HandSolder, F.Cu at (94.5, 72.5)
- added C96: 100nF, Capacitor_SMD:C_1206_3216Metric_Pad1.33x1.80mm_HandSolder, F.Cu at (94.5, 75.9)
- added C97: 220uF, Capacitor_THT:CP_Radial_D6.3mm_P2.50mm, F.Cu at (68.4, 177.7)
- added C98: 100nF, Capacitor_SMD:C_1206_3216Metric_Pad1.33x1.80mm_HandSolder, F.Cu at (88.4, 149.4)
- added C99: 100nF, Capacitor_SMD:C_1206_3216Metric_Pad1.33x1.80mm_HandSolder, F.Cu at (62.5, 175.4)
- added D2: 1N4007, Diode_THT:D_DO-41_SOD81_P10.16mm_Horizontal, F.Cu at (195.6, 45.1)
- added D3: SMAJ400A, Diode_SMD:D_SMA, F.Cu at (85.1, 69.9)
- added D4: 1N4007, Diode_THT:D_DO-41_SOD81_P10.16mm_Horizontal, F.Cu at (195.6, 69.8)
- added FB3: FB, Inductor_SMD:L_1206_3216Metric_Pad1.42x1.75mm_HandSolder, F.Cu at (103.9, 171.4)
- added IC2: TPS7A4901, Custom:TPS7A4901DRBR, F.Cu at (104.5, 159.0)
- added IC4: USBLC6, Package_TO_SOT_SMD:SOT-23-6_Handsoldering, F.Cu at (251.4, 172.7)
- added IC5: ESP32-S3-WROOM-1U-N16R8, Custom:ESP32S3WROOM1UN16R8, F.Cu at (229.0, 169.4)
- added IC6: RESET, Custom:TS026650BK100SCRD, F.Cu at (61.8, 157.8)
- added IC7: BOOT, Custom:TS026650BK100SCRD, F.Cu at (61.8, 166.9)
- added J10: PWR SW, Connector_JST:JST_XH_B2B-XH-A_1x02_P2.50mm_Vertical, F.Cu at (130.3, 35.6)
- added J13: USB-B CONNECTOR, Custom:USBC, F.Cu at (257.4, 171.5)
- added K1: Relay_DPST-NO, Relay_THT:Relay_DPST_Omron_G2RL-2A, F.Cu at (201.0, 43.7)
- added K2: Relay_DPST-NO, Relay_THT:Relay_DPST_Omron_G2RL-2A, F.Cu at (201.0, 68.5)
- added K3: G6K-2P-Y_DC3, G6K:RELAY_G6K-2P-Y_DC3, F.Cu at (148.6, 167.6)
- added K5: G6K-2P-Y_DC3, G6K:RELAY_G6K-2P-Y_DC3, F.Cu at (148.6, 155.6)
- added Q2: 2N7002K, Package_TO_SOT_SMD:SOT-23, F.Cu at (83.5, 65.4)
- added R33: 2K7, Resistor_SMD:R_0805_2012Metric_Pad1.20x1.40mm_HandSolder, F.Cu at (183.5, 103.4)
- added R34: 2K7, Resistor_SMD:R_0805_2012Metric_Pad1.20x1.40mm_HandSolder, F.Cu at (184.5, 93.2)
- added R36: 4R7, Resistor_SMD:R_0805_2012Metric_Pad1.20x1.40mm_HandSolder, F.Cu at (37.0, 123.9)
- added R37: 2R2, Resistor_SMD:R_1206_3216Metric_Pad1.30x1.75mm_HandSolder, F.Cu at (69.3, 123.1)
- added R40: 10K, Resistor_SMD:R_0805_2012Metric_Pad1.20x1.40mm_HandSolder, F.Cu at (174.6, 101.6)
- added R41: 10K, Resistor_SMD:R_0805_2012Metric_Pad1.20x1.40mm_HandSolder, F.Cu at (184.5, 98.3)
- added R53: 22K, Resistor_SMD:R_0805_2012Metric_Pad1.20x1.40mm_HandSolder, F.Cu at (99.8, 75.8)
- added R54: 100R, Resistor_SMD:R_0805_2012Metric_Pad1.20x1.40mm_HandSolder, F.Cu at (72.7, 96.6)
- added R55: 100K, Resistor_SMD:R_0805_2012Metric_Pad1.20x1.40mm_HandSolder, F.Cu at (72.7, 99.5)
- added R56: 22R, Resistor_SMD:R_0603_1608Metric_Pad0.98x0.95mm_HandSolder, F.Cu at (208.5, 173.5)
- added R57: 100K, Resistor_SMD:R_0805_2012Metric_Pad1.20x1.40mm_HandSolder, F.Cu at (253.0, 169.3)
- added R58: 100K, Resistor_SMD:R_0805_2012Metric_Pad1.20x1.40mm_HandSolder, F.Cu at (253.0, 167.3)
- added R59: 22R, Resistor_SMD:R_0603_1608Metric_Pad0.98x0.95mm_HandSolder, F.Cu at (208.5, 175.0)
- added R60: 22R, Resistor_SMD:R_0603_1608Metric_Pad0.98x0.95mm_HandSolder, F.Cu at (208.5, 176.6)
- added R61: 22R, Resistor_SMD:R_0805_2012Metric_Pad1.20x1.40mm_HandSolder, F.Cu at (246.4, 171.4)
- added R62: 22R, Resistor_SMD:R_0805_2012Metric_Pad1.20x1.40mm_HandSolder, F.Cu at (246.4, 173.8)
- added R63: 10K, Resistor_SMD:R_0603_1608Metric_Pad0.98x0.95mm_HandSolder, F.Cu at (81.2, 149.0)
- added R64: 22R, Resistor_SMD:R_0805_2012Metric_Pad1.20x1.40mm_HandSolder, F.Cu at (73.0, 168.8)
- added R65: 22R, Resistor_SMD:R_0805_2012Metric_Pad1.20x1.40mm_HandSolder, F.Cu at (73.0, 171.8)
- added R66: 22R, Resistor_SMD:R_0805_2012Metric_Pad1.20x1.40mm_HandSolder, F.Cu at (77.8, 157.0)
- added R67: 10K, Resistor_SMD:R_0603_1608Metric_Pad0.98x0.95mm_HandSolder, F.Cu at (81.2, 151.5)
- added R70: 100K, Resistor_SMD:R_0805_2012Metric_Pad1.20x1.40mm_HandSolder, F.Cu at (95.9, 175.0)
- added R71: 470R, Resistor_SMD:R_0805_2012Metric_Pad1.20x1.40mm_HandSolder, F.Cu at (191.9, 174.4)
- added R72: 470R, Resistor_SMD:R_0805_2012Metric_Pad1.20x1.40mm_HandSolder, F.Cu at (191.9, 176.4)
- added R73: 1M, Resistor_SMD:R_0805_2012Metric_Pad1.20x1.40mm_HandSolder, F.Cu at (77.8, 165.8)
- added R74: 100K, Resistor_SMD:R_0805_2012Metric_Pad1.20x1.40mm_HandSolder, F.Cu at (98.6, 166.1)
- added R75: 178K, Resistor_SMD:R_0805_2012Metric_Pad1.20x1.40mm_HandSolder, F.Cu at (98.6, 169.1)
- added RV1: R_Potentiometer, Potentiometer_THT:Potentiometer_Alps_RK163_Single_Horizontal, F.Cu at (102.2, 30.6)
- added U10: PCM5102A, Package_SO:TSSOP-20_4.4x6.5mm_P0.65mm, F.Cu at (201.0, 174.6)
- added U11: PCBRCA, Custom:PCBRCA, F.Cu at (263.6, 150.5)
- added U9: LD1117, Package_TO_SOT_SMD:SOT-223-3_TabPin2, F.Cu at (78.5, 177.9)
- C42: value 100nF -> 1uF; footprint Capacitor_SMD:C_1206_3216Metric_Pad1.33x1.80mm_HandSolder -> Capacitor_THT:C_Rect_L7.2mm_W5.5mm_P5.00mm_FKS2_FKP2_MKS2_MKP2
- J5: value IN -> 24V 5A; footprint Connector_JST:JST_XH_B3B-XH-A_1x03_P2.50mm_Vertical -> Custom:CONN_5569-02A_MOL
- moved C89 192.8 mm to (94.5, 62.5)
- moved C90 192.8 mm to (94.5, 65.8)
- moved R19 159.8 mm to (37.0, 112.1), turned to 0 degrees
- moved R20 159.3 mm to (37.0, 115.0), turned to 0 degrees
- moved C37 155.3 mm to (42.4, 119.8), turned to 0 degrees
- moved R17 151.5 mm to (37.0, 106.2), turned to 0 degrees
- moved R18 151.2 mm to (37.0, 109.1), turned to 0 degrees
- moved C67 151.1 mm to (174.9, 97.8), turned to -90 degrees
- moved R44 149.9 mm to (179.5, 105.5), turned to 180 degrees
- moved L4 147.7 mm to (51.0, 134.0), turned to 0 degrees
- moved R45 146.5 mm to (180.5, 91.2), turned to 180 degrees
- moved C36 145.5 mm to (58.3, 135.0)
- moved C32 143.9 mm to (42.4, 109.7), turned to 0 degrees
- moved C25 143.9 mm to (102.6, 128.4), turned to 0 degrees
- moved R22 140.1 mm to (37.0, 120.9)
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Connections:
- net /+5V_MCU renamed /ESP32USB/5V
- net /+5V_PGA_DIG renamed /PGAINPUT/+5V_PGA_DIG
- net /+5V_SYS renamed /POWER SUPPLIES/PVIN
- net /CLIP_LED renamed /MCU/TPA_LED
- net /PGA_CLOCK renamed /MCU/PGA_CLOCK
- net /PGA_CS renamed /MCU/PGA_CS
- net /PGA_DATA renamed /MCU/PGA_DATA
- net /PGA_MUTE renamed /MCU/PGA_MUTE
- net /SWP renamed /POWER SUPPLIES/SWP
- net /TPA_CLIP renamed /MCU/TPA_CLIP
- net /TPA_FAULT renamed /MCU/TPA_FAULT
- net /TPA_RESET renamed /MCU/PGA_RESET
- C21 pad 1: Net-(J5-Pin_1) -> /DACINPUT/PGAIN_R
- C22 pad 1: Net-(J5-Pin_3) -> /DACINPUT/PGAIN_L
- C25 pad 1: /+5V -> /PGAINPUT/+5VA
- C25 pad 2: /-5V -> /PGAINPUT/-5VA
- C30 pad 1: /PVDD_24V -> /POWER SUPPLIES/PVDD_24V
- C31 pad 1: /PVDD_24V -> /POWER SUPPLIES/PVDD_24V
- C35 pad 1: /PVDD_24V -> /POWER SUPPLIES/PVDD_24V
- C36 pad 1: /PVDD_24V -> /POWER SUPPLIES/PVDD_24V
- C41 pad 1: /PVDD_24V -> /POWER SUPPLIES/PVDD_24V
- C42 pad 1: /+5V -> Net-(U7-V_{OUT}L)
- C42 pad 2: /-5V -> /PGAINPUT/VOUTL
- C44 pad 1: /-5V -> /PGAINPUT/-5VA
- C45 pad 1: /+5V -> /PGAINPUT/+5VA
- C48 pad 1: /PVDD_24V -> /POWER SUPPLIES/PVDD_24V
- C49 pad 1: /PVDD_24V -> /POWER SUPPLIES/PVDD_24V
- C68 pad 1: /+12V_OPAMP -> /POWER SUPPLIES/+12V_OPAMP
- C69 pad 1: /+12V_OPAMP -> /POWER SUPPLIES/+12V_OPAMP
- C70 pad 1: /−5VA -> /PGAINPUT/-5VA
- C71 pad 1: /−5VA -> /PGAINPUT/-5VA
- C72 pad 1: /+5VA -> /PGAINPUT/+5VA
- C73 pad 1: /+5VA -> /PGAINPUT/+5VA
- C74 pad 1: /VDD_TPA -> /POWER SUPPLIES/VDD_TPA
- C75 pad 1: /GVDD_AB -> /POWER SUPPLIES/GVDD_AB
- C76 pad 1: /GVDD_CD -> /POWER SUPPLIES/GVDD_CD
- C77 pad 1: /GVDD_CD -> /POWER SUPPLIES/GVDD_CD
- C78 pad 1: /GVDD_AB -> /POWER SUPPLIES/GVDD_AB
- C79 pad 1: /VDD_TPA -> /POWER SUPPLIES/VDD_TPA
- C80 pad 1: /+12V_OPAMP -> /POWER SUPPLIES/+12V_OPAMP
- C85 pad 1: /POT_WIPER -> /MCU/POT_WIPER
- D1 pad 1: /PVDD_24V -> Net-(D1-K)
- F1 pad 2: Net-(F1-Pad2) -> Net-(D3-A1)
- J5 pad 1: Net-(J5-Pin_1) -> Net-(F1-Pad1)
- Q1 pad 2: Net-(Q1-Pad2) -> Net-(D3-A1)
- Q1 pad 3: /PVDD_24V -> Net-(D1-K)
- R21 pad 1: /+5VA -> /PGAINPUT/+5VA
- R22 pad 2: /−5VA -> /PGAINPUT/-5VA
- R39 pad 1: /VOUTL -> /PGAINPUT/VOUTL
- R48 pad 2: /GVDD_AB -> /POWER SUPPLIES/GVDD_AB
- R49 pad 2: /GVDD_CD -> /POWER SUPPLIES/GVDD_CD
- R51 pad 1: /POT_WIPER -> /MCU/POT_WIPER
- R51 pad 2: Net-(J9-Pin_2) -> /MCU/POT_WIPER
- TH1 pad 1: Net-(F1-Pad2) -> Net-(K1-Pad23)
- TH1 pad 2: Net-(Q1-Pad2) -> /POWER SUPPLIES/PVDD_24V
- U1 pad 12: unconnected-(U1-DVDD-Pad12) -> Net-(U1-DVDD)
- U1 pad 16: unconnected-(U1-OC_ADJ-Pad16) -> Net-(U1-OC_ADJ)
- U1 pad 3: unconnected-(U1-VBG-Pad3) -> Net-(U1-VBG)
- U1 pad 9: unconnected-(U1-AVDD-Pad9) -> Net-(U1-AVDD)
- U1 pad V: GND -> (no net)
- U2 pad 11: /POT_WIPER -> /MCU/POT_WIPER
- U2 pad 6: unconnected-(U2-PB3-Pad6) -> /MCU/INRUSH_CTRL
- U3 pad 3: /PVDD_24V -> /POWER SUPPLIES/PVDD_24V
- U3 pad 5: /PVDD_24V -> /POWER SUPPLIES/PVDD_24V
- U6 pad 4: /-5V -> /PGAINPUT/-5VA
- U6 pad 8: /+5V -> /PGAINPUT/+5VA
- U7 pad 12: /+5V -> /PGAINPUT/+5VA
- U7 pad 13: /-5V -> /PGAINPUT/-5VA
- U8 pad 3: /PVDD_24V -> /POWER SUPPLIES/PVDD_24V
- U8 pad 5: /PVDD_24V -> /POWER SUPPLIES/PVDD_24V
Routing:
- net Net-(J10-Pin_1): track 0.00 -> 76.4 mm
- net /POWER SUPPLIES/PVDD_24V: track 0.00 -> 49.3 mm
- net Net-(U7-V_{OUT}L): track 83.1 -> 34.0 mm
- net /PGAINPUT/+5VA: track 0.00 -> 35.6 mm
- net Net-(U7-V_{OUT}R): track 0.00 -> 33.0 mm
- net /DACINPUT/DATA: track 0.00 -> 30.5 mm, vias 0 -> 2
- net /ESP32USB/VBUS-SENSE: track 0.00 -> 30.4 mm, vias 0 -> 2
- net /DACINPUT/LRCK: track 0.00 -> 29.6 mm, vias 0 -> 2
- net /DACINPUT/BCLK: track 0.00 -> 29.4 mm, vias 0 -> 2
- net /PGAINPUT/-5VA: track 0.00 -> 27.6 mm
- net /POWER SUPPLIES/PVIN: track 25.8 -> 0.00 mm, vias 2 -> 0
- net /ESP32USB/D+: track 0.00 -> 17.1 mm
- net Net-(C62-Pad2): track 0.00 -> 16.7 mm
- net Net-(U6B-+): track 4.57 -> 20.5 mm
- net Net-(D1-A): track 0.00 -> 15.6 mm
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- added copper zone on B.Cu, net /POWER SUPPLIES/PVDD_24V
- added copper zone on F.Cu, net Net-(D1-K)
- added copper zone on F.Cu, net Net-(D3-A1)
- added copper zone on B.Cu, net Net-(F1-Pad1)
- added copper zone on B.Cu, net Net-(K1-Pad23)
Other:
- board size 130 x 130 mm -> 152.8 x 155.7 mm
- board text added: "A 2 TPA3250"
- board text added: "Reference"
- board text added: "Series"
