File: TPA3250/TPA3250.kicad_sch (KiCad schematic)
At the start: 167 parts, among them IC3 TPS65133, J1 L +, J2 L -, J3 R +, J4 R -, J5 IN, J6 PROG, J7 24V IN, J8 GND, J9 VOL, Q1 DMP4015SK3, U1 TPA3250, U2 ATtiny1614-SS, U3 LMR51430, U4 OPA1656ID, U5 OPA1656ID, U6 LM4562, U7 PGA2311, U8 LMR51430

Commit message: more work
Parts:
- added C88, C89, C90, C91, C94, C95: 1uF, Capacitor_SMD:C_1206_3216Metric_Pad1.33x1.80mm_HandSolder, symbol Device:C
- added C92, C93: 1000uF, Capacitor_THT:CP_Radial_D12.5mm_P5.00mm, symbol Device:C_Polarized
- added C96: 100nF, Capacitor_SMD:C_1206_3216Metric_Pad1.33x1.80mm_HandSolder, symbol Device:C
- added R53: 22K, Resistor_SMD:R_0805_2012Metric_Pad1.20x1.40mm_HandSolder, symbol Device:R
Connections:
- net GND: now also C88.2, C89.2, C90.2, C91.2, C92.2, C93.2, C94.2, C95.2, C96.2, R53.1
- net PVDD_24V: now also C88.1, C89.1, C90.1, C91.1, C92.1, C93.1
- net at U1.12 (DVDD): now also C95.1
- net at U1.16 (OC_ADJ): now also R53.2
- net at U1.3 (VBG): now also C96.1
- net at U1.9 (AVDD): now also C94.1

Commit message: more work
Parts:
- removed C21, C22, C42, C43: 1uF, Capacitor_THT:C_Rect_L7.2mm_W5.5mm_P5.00mm_FKS2_FKP2_MKS2_MKP2, symbol Device:C
- removed C23, C24: 220pF, Capacitor_SMD:C_0805_2012Metric_Pad1.18x1.45mm_HandSolder, symbol Device:C
- removed C25, C27, C32, C37, C44, C45, C46, C47, C68, C70, C72, C77, C78, C79, C85: 100nF, Capacitor_SMD:C_1206_3216Metric_Pad1.33x1.80mm_HandSolder, symbol Device:C
- removed C26, C28, C29: 10uF, Capacitor_SMD:C_0805_2012Metric_Pad1.18x1.45mm_HandSolder, symbol Device:C
- removed C30: 100-470uF, Capacitor_THT:CP_Radial_D8.0mm_P3.50mm, symbol Device:C_Polarized
- removed C31, C36: 2.2uF, Capacitor_SMD:C_0805_2012Metric_Pad1.18x1.45mm_HandSolder, symbol Device:C
- removed C33, C34, C38, C39, C40: 22uF, Capacitor_SMD:C_1206_3216Metric_Pad1.33x1.80mm_HandSolder, symbol Device:C
- removed C35, C41: 2200uF, Capacitor_THT:CP_Radial_D16.0mm_P7.50mm, symbol Device:C_Polarized
- removed C48, C49, C74, C75, C76, C80, C84, C87: 1uF, Capacitor_SMD:C_1206_3216Metric_Pad1.33x1.80mm_HandSolder, symbol Device:C
- removed C69, C71, C73: 47uF, Capacitor_THT:CP_Radial_D5.0mm_P2.50mm, symbol Device:C_Polarized
- removed C83, C86: 10uF, Capacitor_THT:CP_Radial_D4.0mm_P2.00mm, symbol Device:C_Polarized
- removed D1: ZD 12V, Diode_THT:D_DO-201AD_P12.70mm_Horizontal, symbol Device:D_Zener_Filled
- removed F1: 5A, Fuse:Fuseholder_Cylinder-5x20mm_Stelvio-Kontek_PTF78_Horizontal_Open, symbol Device:Fuse
- removed IC3: TPS65133, Custom:SON45P300X300X80-13N-D, symbol Custom:TPS65133DPDR
- removed J5: IN, Connector_JST:JST_XH_B3B-XH-A_1x03_P2.50mm_Vertical, symbol Connector:Conn_01x03_Socket
- removed J6: PROG, Connector_JST:JST_XH_B3B-XH-A_1x03_P2.50mm_Vertical, symbol Connector:Conn_01x03_Socket
- removed J7: 24V IN, Spade connector:TE_62409-1, symbol Spade connector:62409-1
- removed J8: GND, Spade connector:TE_62409-1, symbol Spade connector:62409-1
- removed J9: VOL, Connector_JST:JST_XH_B3B-XH-A_1x03_P2.50mm_Vertical, symbol Connector:Conn_01x03_Socket
- removed L1, L2: 4.7uH, Inductor_SMD:L_1008_2520Metric_Pad1.43x2.20mm_HandSolder, symbol Device:L
- removed L3: 6.8uH, Custom:SRP6030WA-6R8M, symbol Device:L
- removed L4: 12uH, Custom:SRP6030WA-6R8M, symbol Device:L
- removed Q1: DMP4015SK3, DMP4015SK313, symbol Custom:DMP4015SK3-13
- removed R10, R35, R9: 47K, Resistor_SMD:R_0805_2012Metric_Pad1.20x1.40mm_HandSolder, symbol Device:R
- removed R11, R12: 100R, Resistor_SMD:R_0805_2012Metric_Pad1.20x1.40mm_HandSolder, symbol Device:R
- removed R13, R14, R15, R16: 22R, Resistor_SMD:R_0805_2012Metric_Pad1.20x1.40mm_HandSolder, symbol Device:R
- removed R17, R19: 100K, Resistor_SMD:R_0805_2012Metric_Pad1.20x1.40mm_HandSolder, symbol Device:R
- removed R18: 13K7, Resistor_SMD:R_0805_2012Metric_Pad1.20x1.40mm_HandSolder, symbol Device:R
- removed R20: 5K23, Resistor_SMD:R_0805_2012Metric_Pad1.20x1.40mm_HandSolder, symbol Device:R
- removed R21, R22: 2R2, Resistor_SMD:R_0805_2012Metric_Pad1.20x1.40mm_HandSolder, symbol Device:R
- removed R36: 4R7, Resistor_SMD:R_0805_2012Metric_Pad1.20x1.40mm_HandSolder, symbol Device:R
- removed R37, R48, R49: 2R2, Resistor_SMD:R_1206_3216Metric_Pad1.30x1.75mm_HandSolder, symbol Device:R
- removed R5, R51, R6: 1K, Resistor_SMD:R_0805_2012Metric_Pad1.20x1.40mm_HandSolder, symbol Device:R
- removed R50, R52: 10R, Resistor_SMD:R_0805_2012Metric_Pad1.20x1.40mm_HandSolder, symbol Device:R
- removed R7, R8: 1M, Resistor_SMD:R_0805_2012Metric_Pad1.20x1.40mm_HandSolder, symbol Device:R
- removed TH1: Thermistor_NTC, Resistor_THT:R_Radial_Power_L16.1mm_W9.0mm_P7.37mm, symbol Device:Thermistor_NTC
- removed U2: ATtiny1614-SS, Package_SO:SOIC-14_3.9x8.7mm_P1.27mm, symbol MCU_Microchip_ATtiny:ATtiny1614-SS
- removed U3, U8: LMR51430, Package_TO_SOT_SMD:SOT-23-6_Handsoldering, symbol Regulator_Switching:LMR51430
- removed U6: LM4562, Package_DIP:DIP-8_W7.62mm_Socket, symbol Amplifier_Operational:NE5532
- removed U7: PGA2311, Package_DIP:DIP-16_W7.62mm_Socket, symbol Audio:PGA2310UA
Connections:
- net VOUTL renamed PGAINPUT/VOUTL
- net VOUTR renamed PGAINPUT/VOUTR
Other:
- added sheet DACINPUT (DACINPUT.kicad_sch)
- added sheet ESP32USB (ESP32USB.kicad_sch)
- added sheet MCU (MCU.kicad_sch)
- added sheet PGAINPUT (PGAINPUT.kicad_sch)
- added sheet POWER SUPPLIES (POWER SUPPLIES.kicad_sch)
- added sheet POWERIN (POWERIN.kicad_sch)
- moved on the sheet: C58, C59, C64, C65, C66, C67, C81, C82, C88, C89, C90, C91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
