File: TPA3250/POWERIN.kicad_sch (KiCad schematic)
At the start: 19 parts, among them J10 PWR SW, J5 24V 5A, K1 Relay_DPST-NO, K2 Relay_DPST-NO, Q1 DMP4015SK3, Q2 2N7002K

Commit message: redesign part 1
Parts:
- removed J10: PWR SW, Connector_JST:JST_XH_B2B-XH-A_1x02_P2.50mm_Vertical, symbol Connector:Conn_01x02_Socket
- K1: value Relay_DPST-NO -> STANDBY RELAY
- K2: value Relay_DPST-NO -> INRUSH RELAY
- TH1: value Thermistor_NTC -> 10R NTC; footprint Resistor_THT:R_Radial_Power_L16.1mm_W9.0mm_P7.37mm -> Capacitor_THT:C_Disc_D16.0mm_W5.0mm_P7.50mm
Connections:
- net PWR-SW-1: now reaches K1.A2
