File: PCM3250-SPLIT/DACINPUT.kicad_sch (KiCad schematic)
At the start: 28 parts, among them IC2 TPS7A4901, K3 USB, K5 AUX, U10 PCM5102A, U11 AUX IN

Commit message: redesign part 1
Parts:
- removed U11: AUX IN, Custom:PCBRCA, symbol Custom:PCBRCA
- added J7: AUX IN, Connector_JST:JST_XH_B3B-XH-A_1x03_P2.50mm_Vertical, symbol Connector:Conn_01x03_Socket
Connections:
- net GND: now also J7.2 (Pin_2)
- net at K5.3: now also J7.3 (Pin_3)
- net at K5.6: now also J7.1 (Pin_1)
Changed lines of the file:
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@@
 	(wire
 		(pts
-			(xy 191.77 114.3) (xy 191.77 130.81)
+			(xy 191.77 111.76) (xy 191.77 130.81)
 		)
 		(stroke
@@
 	(wire
 		(pts
-			(xy 180.34 114.3) (xy 191.77 114.3)
-		)
-		(stroke
-			(width 0)
-			(type default)
-		)
-	)
-	(wire
-		(pts
 			(xy 144.78 119.38) (xy 134.62 119.38)
 		)
@@
 	(wire
 		(pts
-			(xy 180.34 109.22) (xy 189.23 109.22)
-		)
-		(stroke
-			(width 0)
-			(type default)
-		)
-	)
-	(wire
-		(pts
 			(xy 110.49 22.86) (xy 110.49 46.99)
 		)
@@
 	(wire
 		(pts
+			(xy 176.53 109.22) (xy 189.23 109.22)
+		)
+		(stroke
+			(width 0)
+			(type default)
+		)
+	)
+	(wire
+		(pts
 			(xy 95.25 157.48) (xy 95.25 167.64)
 		)
@@
 	(wire
 		(pts
-			(xy 190.5 104.14) (xy 190.5 86.36)
+			(xy 190.5 106.68) (xy 190.5 86.36)
 		)
 		(stroke
@@
 	(wire
 		(pts
-			(xy 180.34 104.14) (xy 190.5 104.14)
-		)
-		(stroke
-			(width 0)
-			(type default)
-		)
-	)
-	(wire
-		(pts
 			(xy 134.62 127) (xy 134.62 119.38)
 		)
@@
 	(wire
 		(pts
+			(xy 176.53 111.76) (xy 191.77 111.76)
+		)
+		(stroke
+			(width 0)
+			(type default)
+		)
+	)
+	(wire
+		(pts
 			(xy 113.03 116.84) (xy 113.03 134.62)
 		)
@@
 		(pts
 			(xy 33.02 63.5) (xy 46.99 63.5)
+		)
+		(stroke
+			(width 0)
+			(type default)
+		)
+	)
+	(wire
+		(pts
+			(xy 176.53 106.68) (xy 190.5 106.68)
 		)
 		(stroke
@@
 	)
 	(symbol
-		(lib_id "Custom:PCBRCA")
-		(at 182.88 99.06 0)
-		(mirror x)
-		(unit 1)
-		(exclude_from_sim no)
-		(in_bom yes)
-		(on_board yes)
-		(dnp no)
-		(property "Reference" "U11"
-			(at 166.37 124.46 0)
-			(effects
-				(font
-					(size 1.27 1.27)
-				)
-			)
-		)
-		(property "Value" "AUX IN"
-			(at 166.37 121.92 0)
-			(effects
-				(font
-					(size 1.27 1.27)
-				)
-			)
-		)
-		(property "Footprint" "Custom:PCBRCA"
-			(at 182.88 99.06 0)
-			(effects
-				(font
-					(size 1.27 1.27)
-				)
-				(justify bottom)
-				(hide yes)
-			)
-		)
-		(property "Datasheet" ""
-			(at 182.88 99.06 0)
-			(effects
-				(font
-					(size 1.27 1.27)
-				)
-				(hide yes)
-			)
-		)
-		(property "Description" ""
-			(at 182.88 99.06 0)
-			(effects
-				(font
-					(size 1.27 1.27)
-				)
-				(hide yes)
-			)
-		)
-		(pin "P$3"
-		)
-		(pin "P$1"
-		)
-		(pin "P$2"
-		)
-		(instances
-			(project ""
-				(path "/d0eeeeda-311a-416d-b9f7-ac3b9875c0a9/7b577e16-d4db-4c3c-a8cd-e58ae6d0de99"
-					(reference "U11")
-					(unit 1)
-				)
-			)
-		)
-	)
-	(symbol
 		(lib_id "power:GND")
 		(at 156.21 66.04 0)
@@
 					(unit 1)
 				)
+			)
+		)
+	)
+	(symbol
+		(lib_id "Connector:Conn_01x03_Socket")
+		(at 171.45 109.22 180)
+		(unit 1)
+		(exclude_from_sim no)
+		(in_bom yes)
+		(on_board yes)
+		(dnp no)
+		(fields_autoplaced yes)
+		(property "Reference" "J7"
+			(at 172.085 101.6 0)
+			(effects
+				(font
+					(size 1.27 1.27)
+				)
+			)
+		)
+		(property "Value" "AUX IN"
+			(at 172.085 104.14 0)
+			(effects
+				(font
+					(size 1.27 1.27)
+				)
+			)
+		)
+		(property "Footprint" "Connector_JST:JST_XH_B3B-XH-A_1x03_P2.50mm_Vertical"
+			(at 171.45 109.22 0)
+			(effects
+				(font
+					(size 1.27 1.27)
+				)
+				(hide yes)
+			)
+		)
+		(property "Datasheet" "~"
+			(at 171.45 109.22 0)
+			(effects
+				(font
+					(size 1.27 1.27)
+				)
+				(hide yes)
+			)
+		)
+		(property "Description" "Generic connector, single row, 01x03, script generated"
+			(at 171.45 109.22 0)
+			(effects
+				(font
+					(size 1.27 1.27)
+				)
+				(hide yes)
+			)
+		)
+		(pin "2"
+		)
+		(pin "1"
+		)
+		(pin "3"
+		)
+		(instances
+			(project ""
+				(path "/d0eeeeda-311a-416d-b9f7-ac3b9875c0a9/7b577e16-d4db-4c3c-a8cd-e58ae6d0de99"
+					(reference "J7")
+					(unit 1)
+				)

Commit message: lots of work
Parts:
- removed C101, C115: 10nF, Capacitor_SMD:C_0805_2012Metric_Pad1.18x1.45mm_HandSolder, symbol Device:C
- removed C103, C116: 10uF, Capacitor_SMD:C_1206_3216Metric_Pad1.33x1.80mm_HandSolder, symbol Device:C
- removed IC2: TPS7A4901, Custom:TPS7A4901DRBR, symbol Custom:TPS7A4901DRBR
- removed R56, R59, R60: 22R, Resistor_SMD:R_0603_1608Metric_Pad0.98x0.95mm_HandSolder, symbol Device:R
- removed R74: 100K, Resistor_SMD:R_0805_2012Metric_Pad1.20x1.40mm_HandSolder, symbol Device:R
- removed R75: 178K, Resistor_SMD:R_0805_2012Metric_Pad1.20x1.40mm_HandSolder, symbol Device:R
Connections:
- net BCLK: now also U10.13 (BCK)
- net DATA: now also U10.14 (DIN)
- net LRCK: now also U10.15 (LRCK)
- net 3V3 renamed DAC_3V3
