File: PCM3250-SPLIT/PGAINPUT.kicad_sch (KiCad schematic)
At the start: 24 parts, among them U6 LM4562, U7 PGA2311

Commit message: lots of work
Parts:
- added C120, C123, C124: 47uF, Capacitor_THT:CP_Radial_D5.0mm_P2.50mm, symbol Device:C_Polarized
Connections:
- net +5VA: now also C120.1
- net +5V_PGA_DIG: now also C124.1
- net -5VA: now also C123.2
- net GND: now also C120.2, C123.1, C124.2
