File: PCM3250-SPLIT/POWERIN.kicad_sch (KiCad schematic)
At the start: 19 parts, among them J11 GND, J5 VCC, K1 STANDBY RELAY, K2 INRUSH RELAY, Q1 DMP4015SK3, Q2 2N7002K

Commit message: lots of work
Connections:
- net PVDD_24V: no longer D4.1 (K), K2.A1
- net at K1.23, K2.24, TH1.1: now also D4.1 (K), K2.A1
Changed lines of the file:
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@@
 	(paper "A4")
 	(junction
-		(at 180.34 86.36)
-		(diameter 0)
-		(color 0 0 0 0)
-	)
-	(junction
 		(at 201.93 68.58)
 		(diameter 0)
@@
 	)
 	(junction
+		(at 151.13 83.82)
+		(diameter 0)
+		(color 0 0 0 0)
+	)
+	(junction
 		(at 236.22 68.58)
 		(diameter 0)
@@
 	(wire
 		(pts
+			(xy 151.13 83.82) (xy 151.13 106.68)
+		)
+		(stroke
+			(width 0)
+			(type default)
+		)
+	)
+	(wire
+		(pts
 			(xy 151.13 68.58) (xy 161.29 68.58)
 		)
@@
 	(wire
 		(pts
-			(xy 180.34 91.44) (xy 180.34 86.36)
-		)
-		(stroke
-			(width 0)
-			(type default)
-		)
-	)
-	(wire
-		(pts
 			(xy 181.61 118.11) (xy 181.61 120.65)
 		)
@@
 	(wire
 		(pts
-			(xy 151.13 106.68) (xy 151.13 91.44)
+			(xy 151.13 68.58) (xy 151.13 83.82)
 		)
 		(stroke
@@
 	(wire
 		(pts
-			(xy 151.13 68.58) (xy 151.13 83.82)
-		)
-		(stroke
-			(width 0)
-			(type default)
-		)
-	)
-	(wire
-		(pts
 			(xy 252.73 68.58) (xy 261.62 68.58)
 		)
@@
 		)
 		(stroke
-			(width 0)
-			(type default)
-		)
-	)
-	(wire
-		(pts
-			(xy 151.13 91.44) (xy 180.34 91.44)
-		)
-		(stroke
