File: PCM3250-SPLIT/PCM3250-SPLIT.kicad_pcb (KiCad board)
At the start: 4 copper layers, 152.8 x 155.7 mm, 248 parts, among them IC2 TPS7A4901, IC3 TPS65133, IC4 USBLC6, IC5 ESP32-S3-WROOM-1U-N16R8, IC6 RESET, IC7 BOOT, J1 L +, J13 USB IN, J2 L -, J3 R +, J4 R -, J5 24V 5A, J6 PROG, J8 FRONT PANEL, K1 STANDBY RELAY, K2 INRUSH RELAY, K3 USB, K5 AUX, Q1 DMP4015SK3, Q2 2N7002K, U1 TPA3250, U10 PCM5102A, U11 AUX IN, U12 ULN2003A, U13 LD1117, U14 ATtiny1616, U3 LMR51430, U4 OPA1656ID, U5 OPA1656ID, U6 LM4562, U7 PGA2311, U8 LMR51430, U9 LD1117

Commit message: redesign part 1
Parts:
- removed U11: AUX IN, Custom:PCBRCA
- added AMP1: POWER 2, Connector_JST:JST_XH_B8B-XH-A_1x08_P2.50mm_Vertical, F.Cu at (108.6, 69.5)
- added AMP2: POWER 1, Connector_JST:JST_XH_B8B-XH-A_1x08_P2.50mm_Vertical, F.Cu at (84.5, 121.7)
- added H5: MountingHole, MountingHole:MountingHole_4.3mm_M4, F.Cu at (219.6, 34.4)
- added H6: MountingHole, MountingHole:MountingHole_4.3mm_M4, F.Cu at (130.3, 34.5)
- added H7: MountingHole, MountingHole:MountingHole_4.3mm_M4, F.Cu at (130.3, 146.8)
- added H8: MountingHole, MountingHole:MountingHole_4.3mm_M4, F.Cu at (219.6, 146.8)
- added J10: POWER 2, Connector_JST:JST_XH_B8B-XH-A_1x08_P2.50mm_Vertical, F.Cu at (42.9, 167.5)
- added J11: GND, Spade connector:TE_62409-1, F.Cu at (216.4, 51.1)
- added J7: AUX IN, Connector_JST:JST_XH_B3B-XH-A_1x03_P2.50mm_Vertical, F.Cu at (32.5, 35.9)
- added J9: POWER 1, Connector_JST:JST_XH_B8B-XH-A_1x08_P2.50mm_Vertical, F.Cu at (164.4, 145.4)
- J5: value 24V 5A -> VCC; footprint Custom:CONN_5569-02A_MOL -> Spade connector:TE_62409-1
- moved C101 409.0 mm to (457.0, 198.6)
- moved C106 409.0 mm to (425.7, 234.9)
- moved C107 409.0 mm to (425.7, 238.2)
- moved C112 409.0 mm to (457.0, 207.7)
- moved C115 409.0 mm to (457.0, 210.7)
- moved C68 409.0 mm to (454.6, 164.3)
- moved FB3 409.0 mm to (467.1, 220.9)
- moved C104 409.0 mm to (496.4, 192.6)
- moved C105 409.0 mm to (496.4, 195.9)
- moved C109 409.0 mm to (451.6, 208.9)
- moved C113 409.0 mm to (465.1, 230.6)
- moved C114 409.0 mm to (465.1, 233.9)
- moved C69 409.0 mm to (447.7, 172.6)
- moved C74 409.0 mm to (460.6, 157.6)
- moved C75 409.0 mm to (460.6, 160.9)
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Connections:
- J5 pad 2: GND -> Net-(F1-Pad1)
Routing:
- net /ESP32USB/5V: track 275.3 -> 89.5 mm
- net Net-(J7-Pin_3): track 143.4 -> 0.00 mm
- net Net-(J7-Pin_1): track 132.0 -> 0.01 mm
- net /PWR-SW-1: track 79.5 -> 0.00 mm
- net /PVDD_24V: track 108.4 -> 57.0 mm
- net Net-(C118-Pad1): track 52.2 -> 4.55 mm
- net Net-(C117-Pad1): track 52.1 -> 4.53 mm
- net /PGAINPUT/+5V_PGA_DIG: track 75.2 -> 28.5 mm
- net /MCU/PGA_MUTE: track 44.8 -> 0.04 mm, vias 2 -> 1
- net Net-(U7-V_{OUT}R): track 40.9 -> 0.00 mm
- net /MCU/PGA_CLOCK: track 38.4 -> 0.00 mm, vias 2 -> 0
- net Net-(D1-K): track 37.0 -> 0.00 mm
- net /ESP32USB/EN: track 47.6 -> 12.2 mm
- net /MCU/PGA_DATA: track 33.7 -> 0.00 mm, vias 2 -> 0
- net Net-(U7-V_{OUT}L): track 33.4 -> 0.00 mm
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- added copper zone on B.Cu, net GND
- removed copper zone on B.Cu, net /PVDD_24V
- removed copper zone on F.Cu, net Net-(D1-K)
- removed copper zone on F.Cu, net Net-(D3-A1)
- removed copper zone on B.Cu, net Net-(F1-Pad1)
- removed copper zone on B.Cu, net Net-(K1-Pad23)
Other:
- board size 152.8 x 155.7 mm -> 209.7 x 123.5 mm

Commit message: lots of work
Parts:
- removed the C88 at (64.9, 88.0)
- removed the C88 at (64.9, 102.4)
- removed the C91 at (65.7, 99.9)
- removed the C91 at (65.7, 90.5)
- removed C93: 1000uF, Capacitor_THT:CP_Radial_D12.5mm_P5.00mm
- removed R64, R65, R66: 22R, Resistor_SMD:R_0805_2012Metric_Pad1.20x1.40mm_HandSolder
- added C116: 10uF, Capacitor_SMD:C_1206_3216Metric_Pad1.33x1.80mm_HandSolder, F.Cu at (258.8, 107.6)
- added C120: 47uF, Capacitor_THT:CP_Radial_D5.0mm_P2.50mm, F.Cu at (37.3, 56.4)
- added C123: 47uF, Capacitor_THT:CP_Radial_D5.0mm_P2.50mm, F.Cu at (37.3, 75.4)
- added C124: 47uF, Capacitor_THT:CP_Radial_D5.0mm_P2.50mm, F.Cu at (63.8, 51.6)
- added C88: 1uF, Capacitor_SMD:C_1206_3216Metric_Pad1.33x1.80mm_HandSolder, F.Cu at (64.9, 104.6)
- added C91: 1uF, Capacitor_SMD:C_1206_3216Metric_Pad1.33x1.80mm_HandSolder, F.Cu at (65.7, 102.1)
- added G***: LOGO, Custom:LOGONEW, F.Cu at (266.6, 46.0)
- added J12: VOL, Connector_JST:JST_XH_B3B-XH-A_1x03_P2.50mm_Vertical, F.Cu at (67.1, 34.8)
- added J14: POWER BOARD CONNECTOR 3, Connector_JST:JST_XH_B6B-XH-A_1x06_P2.50mm_Vertical, F.Cu at (126.7, 126.0)
- added J15: AMP BOARD CONNECTOR 3, Connector_JST:JST_XH_B6B-XH-A_1x06_P2.50mm_Vertical, F.Cu at (58.2, 123.4)
- added R74: 100K, Resistor_SMD:R_0805_2012Metric_Pad1.20x1.40mm_HandSolder, F.Cu at (271.0, 104.1)
- added R75: 178K, Resistor_SMD:R_0805_2012Metric_Pad1.20x1.40mm_HandSolder, F.Cu at (271.0, 107.1)
- AMP1: value POWER 2 -> AMP BOARD CONNECTOR 1
- AMP2: value POWER 1 -> AMP BOARD CONNECTOR 2
- J10: value POWER 2 -> POWER BOARD CONNECTOR 2
- J8: value FRONT PANEL -> POWER SW; footprint Connector_JST:JST_XH_B8B-XH-A_1x08_P2.50mm_Vertical -> Connector_JST:JST_XH_B2B-XH-A_1x02_P2.50mm_Vertical
- J9: value POWER 1 -> POWER BOARD CONNECTOR 1
- moved C82 444.3 mm to (24.6, 82.0), turned to 180 degrees
- moved C81 441.0 mm to (26.2, 117.9), turned to 180 degrees
- moved R53 425.1 mm to (38.8, 99.7)
- moved C95 415.1 mm to (43.3, 98.0), turned to 180 degrees
- moved C94 415.1 mm to (43.3, 95.6), turned to 180 degrees
- moved C114 405.8 mm to (102.2, 52.2)
- moved C113 405.4 mm to (102.2, 49.8)
- moved FB3 403.6 mm to (106.0, 40.8), turned to 180 degrees
- moved R70 397.5 mm to (105.4, 42.9)
- moved C109 396.4 mm to (94.4, 37.1), turned to 90 degrees
- moved C90 393.8 mm to (64.7, 90.5), turned to 45 degrees
- moved C89 392.5 mm to (65.7, 92.8), turned to 45 degrees
- moved C108 390.3 mm to (93.7, 49.8), turned to 180 degrees
- moved C98 385.4 mm to (101.7, 37.2), turned to 90 degrees
- moved C112 382.0 mm to (110.7, 46.2), turned to 180 degrees
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Connections:
- net /DACINPUT/DATA renamed /DATA-P
- AMP1 pad 1: unconnected-(AMP1-Pin_1-Pad1) -> /BCLK-A
- AMP1 pad 2: unconnected-(AMP1-Pin_2-Pad2) -> GND
- AMP1 pad 3: unconnected-(AMP1-Pin_3-Pad3) -> /DATA-A
- AMP1 pad 4: unconnected-(AMP1-Pin_4-Pad4) -> GND
- AMP1 pad 5: unconnected-(AMP1-Pin_5-Pad5) -> /LRCK-A
- AMP1 pad 6: unconnected-(AMP1-Pin_6-Pad6) -> GND
- AMP1 pad 7: unconnected-(AMP1-Pin_7-Pad7) -> /DAC_3V3-A
- AMP1 pad 8: unconnected-(AMP1-Pin_8-Pad8) -> GND
- AMP2 pad 1: unconnected-(AMP2-Pin_1-Pad1) -> /-5VA-A
- AMP2 pad 2: unconnected-(AMP2-Pin_2-Pad2) -> GND
- AMP2 pad 3: unconnected-(AMP2-Pin_3-Pad3) -> /+5VA-A
- AMP2 pad 4: unconnected-(AMP2-Pin_4-Pad4) -> /+5V_PGA_DIG-A
- AMP2 pad 5: unconnected-(AMP2-Pin_5-Pad5) -> GND
- AMP2 pad 6: unconnected-(AMP2-Pin_6-Pad6) -> /+5V_MCU-A
- AMP2 pad 7: unconnected-(AMP2-Pin_7-Pad7) -> GND
- AMP2 pad 8: unconnected-(AMP2-Pin_8-Pad8) -> /INRUSH_CTRL-A
- C103 pad 2: /DACINPUT/+5V_SYS -> /POWER SUPPLIES/+5V_SYS
- C108 pad 1: /DACINPUT/3V3 -> /DAC_3V3-A
- C109 pad 1: /DACINPUT/3V3 -> /DAC_3V3-A
- C112 pad 1: /DACINPUT/3V3 -> /DAC_3V3-A
- C115 pad 2: /DACINPUT/3V3 -> /DAC_3V3-P
- C121 pad 1: /ESP32USB/5V -> /+5V_MCU-A
- C25 pad 1: /PGAINPUT/+5VA -> /+5VA-A
- C25 pad 2: /PGAINPUT/-5VA -> /-5VA-A
- C44 pad 1: /PGAINPUT/-5VA -> /-5VA-A
- C45 pad 1: /PGAINPUT/+5VA -> /+5VA-A
- C47 pad 1: /PGAINPUT/+5V_PGA_DIG -> /+5V_PGA_DIG-A
- C68 pad 1: /POWER SUPPLIES/+12V_OPAMP -> /+12V_OPAMP
- C69 pad 1: /POWER SUPPLIES/+12V_OPAMP -> /+12V_OPAMP
- C70 pad 1: /PGAINPUT/-5VA -> /-5VA-P
- C71 pad 1: /PGAINPUT/-5VA -> /-5VA-P
- C72 pad 1: /PGAINPUT/+5VA -> /+5VA-P
- C73 pad 1: /PGAINPUT/+5VA -> /+5VA-P
- C80 pad 1: /POWER SUPPLIES/+12V_OPAMP -> /+12V_OPAMP
- C83 pad 1: /ESP32USB/5V -> /+5V_MCU-P
- C84 pad 1: /ESP32USB/5V -> /+5V_MCU-P
- C86 pad 1: /PGAINPUT/+5V_PGA_DIG -> /+5V_PGA_DIG-P
- C87 pad 1: /PGAINPUT/+5V_PGA_DIG -> /+5V_PGA_DIG-P
- C97 pad 1: /ESP32USB/5V -> /+5V_MCU-P
- C99 pad 1: /ESP32USB/5V -> /+5V_MCU-P
- D4 pad 1: /PVDD_24V -> Net-(D4-K)
- FB3 pad 1: /DACINPUT/3V3 -> /DAC_3V3-A
- IC2 pad 1: /DACINPUT/3V3 -> /DAC_3V3-P
- IC2 pad 5: /DACINPUT/+5V_SYS -> /POWER SUPPLIES/+5V_SYS
- IC2 pad 8: /DACINPUT/+5V_SYS -> /POWER SUPPLIES/+5V_SYS
- IC5 pad 4: /DACINPUT/BCLK -> /BCLK-P
- IC5 pad 5: /DACINPUT/LRCK -> /LRCK-P
- J10 pad 1: unconnected-(J10-Pin_1-Pad1) -> /-5VA-P
- J10 pad 2: unconnected-(J10-Pin_2-Pad2) -> GND
- J10 pad 3: unconnected-(J10-Pin_3-Pad3) -> /+5VA-P
- J10 pad 4: unconnected-(J10-Pin_4-Pad4) -> /+5V_PGA_DIG-P
- J10 pad 5: unconnected-(J10-Pin_5-Pad5) -> GND
- J10 pad 6: unconnected-(J10-Pin_6-Pad6) -> /+5V_MCU-P
- J10 pad 7: unconnected-(J10-Pin_7-Pad7) -> GND
- J10 pad 8: unconnected-(J10-Pin_8-Pad8) -> /INRUSH_CTRL-P
- J9 pad 1: unconnected-(J9-Pin_1-Pad1) -> Net-(J9-Pin_1)
- J9 pad 2: unconnected-(J9-Pin_2-Pad2) -> GND
- J9 pad 3: unconnected-(J9-Pin_3-Pad3) -> Net-(J9-Pin_3)
- J9 pad 4: unconnected-(J9-Pin_4-Pad4) -> GND
- J9 pad 5: unconnected-(J9-Pin_5-Pad5) -> Net-(J9-Pin_5)
- J9 pad 6: unconnected-(J9-Pin_6-Pad6) -> GND
- J9 pad 7: unconnected-(J9-Pin_7-Pad7) -> /DAC_3V3-P
- J9 pad 8: unconnected-(J9-Pin_8-Pad8) -> GND
- K1 pad 23: Net-(K1-Pad23) -> Net-(D4-K)
- K2 pad 24: Net-(K1-Pad23) -> Net-(D4-K)
- K2 pad A1: /PVDD_24V -> Net-(D4-K)
- R21 pad 1: /PGAINPUT/+5VA -> /+5VA-P
- R22 pad 2: /PGAINPUT/-5VA -> /-5VA-P
- R36 pad 2: /POWER SUPPLIES/+12V_OPAMP -> /+12V_OPAMP
- R50 pad 2: /ESP32USB/5V -> /+5V_MCU-P
- R52 pad 2: /PGAINPUT/+5V_PGA_DIG -> /+5V_PGA_DIG-P
- R54 pad 2: /MCU/INRUSH_CTRL -> /INRUSH_CTRL-P
- R56 pad 1: Net-(U10-LRCK) -> Net-(J9-Pin_1)
- R56 pad 2: /DACINPUT/LRCK -> /BCLK-P
- R59 pad 1: Net-(U10-DIN) -> Net-(J9-Pin_3)
- R60 pad 1: Net-(U10-BCK) -> Net-(J9-Pin_5)
- R60 pad 2: /DACINPUT/BCLK -> /LRCK-P
- TH1 pad 1: Net-(K1-Pad23) -> Net-(D4-K)
- U10 pad 1: /DACINPUT/3V3 -> /DAC_3V3-A
- U10 pad 13: Net-(U10-BCK) -> /BCLK-A
- U10 pad 14: Net-(U10-DIN) -> /DATA-A
- U10 pad 15: Net-(U10-LRCK) -> /LRCK-A
- U10 pad 8: /DACINPUT/3V3 -> /DAC_3V3-A
- U12 pad 9: /ESP32USB/5V -> /+5V_MCU-A
- U13 pad 3: /ESP32USB/5V -> /+5V_MCU-A
- U14 pad 8: /MCU/INRUSH_CTRL -> /INRUSH_CTRL-A
- U6 pad 4: /PGAINPUT/-5VA -> /-5VA-A
- U6 pad 8: /PGAINPUT/+5VA -> /+5VA-A
- U7 pad 1: /PGAINPUT/+5V_PGA_DIG -> /+5V_PGA_DIG-A
- U7 pad 12: /PGAINPUT/+5VA -> /+5VA-A
- U7 pad 13: /PGAINPUT/-5VA -> /-5VA-A
- U7 pad 4: /PGAINPUT/+5V_PGA_DIG -> /+5V_PGA_DIG-A
- U9 pad 3: /ESP32USB/5V -> /+5V_MCU-P
Routing:
- net /ESP32USB/5V: track 89.5 -> 0.00 mm, vias 3 -> 0
- net /+5VA-A: track 0.00 -> 67.9 mm, vias 0 -> 2
- net Net-(C117-Pad1): track 4.53 -> 72.0 mm
- net Net-(C118-Pad1): track 4.55 -> 66.8 mm
- net Net-(U7-V_{OUT}L): track 0.00 -> 60.8 mm
- net /-5VA-A: track 0.00 -> 58.0 mm, vias 0 -> 1
- net /VOL-3V3: track 56.3 -> 111.9 mm, vias 1 -> 3
- net /+5V_PGA_DIG-A: track 0.00 -> 54.6 mm
- net Net-(D1-K): track 0.00 -> 54.1 mm
- net Net-(U7-V_{OUT}R): track 0.00 -> 50.8 mm
- net /INRUSH_CTRL-A: track 0.00 -> 46.3 mm, vias 0 -> 2
- net /+5V_MCU-A: track 0.00 -> 45.3 mm, vias 0 -> 1
- net /PGAINPUT/+5VA: track 42.3 -> 0.00 mm, vias 1 -> 0
- net /ESP32USB/EN: track 12.2 -> 54.4 mm, vias 1 -> 2
- net /DAC_3V3-A: track 0.00 -> 41.0 mm
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- added copper zone on B.Cu, net /PVDD_24V
- added copper zone on F.Cu, net Net-(D1-K)
- added copper zone on F.Cu, net Net-(D3-A1)
Other:
- board size 209.7 x 123.5 mm -> 229.9 x 123.5 mm
- board text added: "GND W 3V3"
- board text added: "P 3V3 G"
- board text added: "R G L"
- board text added: "TPA3250 Class-D Amplifier With PFFB Amplifier Board PGA2311 Volume Control Tom Watson Audio - 2026"
- board text added: "TPA3250 Class-D Amplifier With PFFB Power Supply PGA2311 Volume Control Tom Watson Audio - 2026"
- board text removed: "A 2"
- board text removed: "GND 3V3 P"
- board text removed: "INPUT-GND"
- board text removed: "INPUT-MCU"
- board text removed: "NC"
- board text removed: "PWR-GND"
- board text removed: "PWR-RLY"
- board text removed: "TPA3250"
- board text removed: "TPA3250 Class-D Amplifier With PFFB PGA2311 Volume Control Tom Watson Audio - 2026"
- board text removed: "VOL-3V3"
- board text removed: "VOL-GND"
- board text removed: "VOL-WIPER"

Commit message: more work
Parts:
- added C93: 1000uF, Capacitor_THT:CP_Radial_D12.5mm_P5.00mm, F.Cu at (64.0, 117.7)
- moved C77 221.7 mm to (48.4, 106.2), turned to -90 degrees
- moved C76 217.8 mm to (46.0, 106.2), turned to -90 degrees
- moved C78 216.5 mm to (52.2, 105.9)
- moved C75 209.4 mm to (52.2, 108.3)
- moved C79 201.9 mm to (51.9, 88.9)
- moved C74 196.1 mm to (51.9, 86.5)
- moved J15 26.4 mm to (84.7, 123.4)
- moved C92 0.40 mm to (47.5, 117.6)
Connections:
- C74 pad 1: /POWER SUPPLIES/VDD_TPA -> /GVDD_AB-A
- C75 pad 1: /POWER SUPPLIES/GVDD_AB -> /GVDD_CD-A
- C76 pad 1: /POWER SUPPLIES/GVDD_CD -> /VDD_TPA-A
- C77 pad 1: /POWER SUPPLIES/GVDD_CD -> /VDD_TPA-A
- C78 pad 1: /POWER SUPPLIES/GVDD_AB -> /GVDD_CD-A
- C79 pad 1: /POWER SUPPLIES/VDD_TPA -> /GVDD_AB-A
- J15 pad 1: unconnected-(J15-Pin_1-Pad1) -> /GVDD_CD-A
- J15 pad 2: unconnected-(J15-Pin_2-Pad2) -> GND
- J15 pad 3: unconnected-(J15-Pin_3-Pad3) -> /VDD_TPA-A
- J15 pad 4: unconnected-(J15-Pin_4-Pad4) -> GND
- J15 pad 5: unconnected-(J15-Pin_5-Pad5) -> /GVDD_AB-A
- J15 pad 6: unconnected-(J15-Pin_6-Pad6) -> GND
- R48 pad 2: /POWER SUPPLIES/GVDD_AB -> /POWER SUPPLIES/GVDD_TPA
- U1 pad 1: /GVDD_CD -> /GVDD_AB-A
- U1 pad 21: /VDD_TPA -> /VDD_TPA-A
- U1 pad 22: /GVDD_AB -> /GVDD_CD-A
Routing:
- net /GVDD_AB-A: track 0.00 -> 75.3 mm, vias 0 -> 2
- net /VDD_TPA-A: track 0.00 -> 58.9 mm
- net /GVDD_CD-A: track 0.00 -> 48.0 mm
- net Net-(C12-Pad2): track 46.7 -> 0.10 mm
- net Net-(C13-Pad1): track 46.1 -> 0.03 mm
- net Net-(C1-Pad2): track 45.7 -> 0.03 mm
- net Net-(C11-Pad1): track 46.4 -> 5.40 mm
- net /+12V_OPAMP: track 17.2 -> 50.8 mm, vias 0 -> 3
- net /+5VA-A: track 67.9 -> 58.0 mm
- net /-5VA-A: track 58.0 -> 56.1 mm
- net Net-(U7-V_{OUT}L): track 60.8 -> 59.5 mm
- net /VOL-3V3: track 111.9 -> 110.7 mm
- net /+5V_PGA_DIG-A: track 54.6 -> 53.7 mm
- net Net-(U7-V_{OUT}R): track 50.8 -> 50.3 mm
- added copper zone on F.Cu, net Net-(C1-Pad2)
- added copper zone on F.Cu, net Net-(C11-Pad1)
- added copper zone on F.Cu, net Net-(C12-Pad2)
- added copper zone on F.Cu, net Net-(C13-Pad1)
