File: PCM3250-SPLIT/PCM3250-SPLIT.kicad_sch (KiCad schematic)
At the start: 90 parts, among them J1 L +, J2 L -, J3 R +, J4 R -, J8 FRONT PANEL, U1 TPA3250, U4 OPA1656ID, U5 OPA1656ID

Commit message: redesign part 1
Parts:
- added AMP1, J10: POWER 2, Connector_JST:JST_XH_B8B-XH-A_1x08_P2.50mm_Vertical, symbol Connector:Conn_01x08_Socket
- added AMP2, J9: POWER 1, Connector_JST:JST_XH_B8B-XH-A_1x08_P2.50mm_Vertical, symbol Connector:Conn_01x08_Socket
- added H5, H6, H7, H8: MountingHole, MountingHole:MountingHole_4.3mm_M4, symbol Mechanical:MountingHole

Commit message: lots of work
Parts:
- removed C93: 1000uF, Capacitor_THT:CP_Radial_D12.5mm_P5.00mm, symbol Device:C_Polarized
- removed J8: FRONT PANEL, Connector_JST:JST_XH_B8B-XH-A_1x08_P2.50mm_Vertical, symbol Connector:Conn_01x08_Socket
- added J12: VOL, Connector_JST:JST_XH_B3B-XH-A_1x03_P2.50mm_Vertical, symbol Connector:Conn_01x03_Socket
- added J14: POWER BOARD CONNECTOR 3, Connector_JST:JST_XH_B6B-XH-A_1x06_P2.50mm_Vertical, symbol Connector:Conn_01x06_Socket
- added J15: AMP BOARD CONNECTOR 3, Connector_JST:JST_XH_B6B-XH-A_1x06_P2.50mm_Vertical, symbol Connector:Conn_01x06_Socket
- added J8: POWER SW, Connector_JST:JST_XH_B2B-XH-A_1x02_P2.50mm_Vertical, symbol Connector:Conn_01x02_Socket
- added R56, R59, R60: 22R, Resistor_SMD:R_0603_1608Metric_Pad0.98x0.95mm_HandSolder, symbol Device:R
- AMP1: value POWER 2 -> AMP BOARD CONNECTOR 1
- AMP2: value POWER 1 -> AMP BOARD CONNECTOR 2
- J10: value POWER 2 -> POWER BOARD CONNECTOR 2
- J9: value POWER 1 -> POWER BOARD CONNECTOR 1
Connections:
- net GND: now also AMP1.2 (Pin_2), AMP1.4 (Pin_4), AMP1.6 (Pin_6), AMP1.8 (Pin_8), AMP2.2 (Pin_2), AMP2.5 (Pin_5), AMP2.7 (Pin_7), J10.2 (Pin_2), J10.5 (Pin_5), J10.7 (Pin_7), J9.2 (Pin_2), J9.4 (Pin_4), J9.6 (Pin_6), J9.8 (Pin_8), J12.1 (Pin_1)
- net PWR-SW-1: now also J8.1 (Pin_1)
- net PWR-SW-2: now also J8.2 (Pin_2)
- net VOL-3V3: now also J12.3 (Pin_3)
- net VOL-WIPER: now also J12.2 (Pin_2)
- net -5VA-P: now reaches J10.1 (Pin_1)
- net +5VA-P: now reaches J10.3 (Pin_3)
- net +5V_PGA_DIG-P: now reaches J10.4 (Pin_4)
- net +5V_MCU-P: now reaches J10.6 (Pin_6)
- net INRUSH_CTRL-P: now reaches J10.8 (Pin_8)
- net BCLK-A: now reaches AMP1.1 (Pin_1)
- net DATA-A: now reaches AMP1.3 (Pin_3)
- net LRCK-A: now reaches AMP1.5 (Pin_5)
- net DAC_3V3-A: now reaches AMP1.7 (Pin_7)
- net -5VA-A: now reaches AMP2.1 (Pin_1)
- net +5VA-A: now reaches AMP2.3 (Pin_3)
- net +5V_PGA_DIG-A: now reaches AMP2.4 (Pin_4)
- net +5V_MCU-A: now reaches AMP2.6 (Pin_6)
- net INRUSH_CTRL-A: now reaches AMP2.8 (Pin_8)
- net at J9.1 (Pin_1): now also R56.1
- net at J9.3 (Pin_3): now also R59.1
- net at J9.5 (Pin_5): now also R60.1
- net DAC_3V3-P: now reaches J9.7 (Pin_7)
- new net BCLK-P: R56.2
- new net DATA-P: R59.2
- new net LRCK-P: R60.2
Other:
- sheet DACINPUT ports: added DAC_3V3; removed none
- sheet POWER SUPPLIES ports: added DAC_3V3; removed +5V_SYS
- moved on the sheet: AMP1, AMP2, J10, J9

Commit message: more work
Parts:
- added C74, C75, C76: 1uF, Capacitor_SMD:C_1206_3216Metric_Pad1.33x1.80mm_HandSolder, symbol Device:C
- added C77, C78, C79: 100nF, Capacitor_SMD:C_1206_3216Metric_Pad1.33x1.80mm_HandSolder, symbol Device:C
- added C93: 1000uF, Capacitor_THT:CP_Radial_D12.5mm_P5.00mm, symbol Device:C_Polarized
Connections:
- net GVDD_AB is gone; now on net GVDD_CD-A: U1.22 (GVDD_AB)
- net GVDD_CD is gone; now on net GVDD_AB-A: U1.1 (GVDD_CD)
- net VDD_TPA is gone; now on net VDD_TPA-A: U1.21 (VDD)
- net GND: now also J15.2 (Pin_2), J15.4 (Pin_4), J15.6 (Pin_6), C74.2, C75.2, C76.2, C77.2, C78.2, C79.2, C93.2
- net PVDD_24V: now also C93.1
- net GVDD_CD-A: now reaches J15.1 (Pin_1)
- net GVDD_CD-A: now also C75.1, C78.1
- net VDD_TPA-A: now reaches J15.3 (Pin_3)
- net VDD_TPA-A: now also C76.1, C77.1
- net GVDD_AB-A: now reaches J15.5 (Pin_5)
- net GVDD_AB-A: now also C74.1, C79.1
Other:
- sheet POWER SUPPLIES ports: added +5V_SYS, GVDD_CD, GVDD_TPA, VDD_TPA; removed none
